File: Stepper Motor Controller/Electrical/Stepper_Motor_Controller.sch (KiCad schematic (older format))
At the start: 69 parts, among them J1 UPDI Header, J2 Stepper Connector, J3 Comm Connector, J4 Comm Connector, U1 AVR32DA32, U2 DRV8825, U3 PER231-P19-N0010, U4 SN74LVC2G17DBVR, U5 UA78M33CKVURG3

Commit message: Added annotations
Other:
- note added: "Connectors to controller and other motors."
- note added: "Microcontroller"
- note added: "Rotatry Encoder"
- note added: "Stepper Motor Driver"
- note added: "Voltage Regulator"
- moved on the sheet: C1, C10, C11, C12, C13, C14, C15, C2, C3, C4, C7, C8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
